File: BLENDER V2.1.kicad_sch (KiCad schematic)
At the start: 32 parts, among them J1 +9V, J2 GND, J3 SEND, J4 IN, J5 RETURN, J6 TO VOLUME POT, J7 OUT, Q1 2SK303, U1 NJM5532

Commit message: v2.1
Parts:
- removed C3: 22u, My_Parts:CP_5mm, symbol Device:C_Polarized
- removed C5: 2.2u, My_Parts:CP_5mm, symbol Device:C_Polarized
- removed J5: RETURN, My_Parts:Header_Pin_1p_Large, symbol Connector:Conn_01x01_Female
- removed R3: 12k, My_Parts:R_Normal, symbol Device:R
- removed RV2: 50kB, My_Parts:POT_ON_BOARD_REVERSE, symbol Device:R_Potentiometer
- added C3: 0.1u, My_Parts:C_Poly_8mm, symbol Device:C
- added C4: 2.2u, My_Parts:CP_5mm, symbol Device:C_Polarized
- added Q2: 2SK303, My_Parts:FET_GSD, symbol Device:Q_NJFET_GSD
- added R4: 1M, My_Parts:R_Normal, symbol Device:R
- added R6: 3k3, My_Parts:R_Normal, symbol Device:R
- J1: value +9V -> 9V
- J3: value SEND -> Virtual GND
- J6: value TO VOLUME POT -> RETURN
- POT1: renamed from RV1; value 10kB -> 10k; footprint My_Parts:POT_ON_BOARD_REVERSE -> My_Parts:Header_Pin_3p
- Q1: footprint My_Parts:FET_GSD2 -> My_Parts:FET_GSD
- R2: value 12k -> 1M
- renumbered C4 to C5, J4 to J5, R9 to R10, R10 to R11, R11 to R12, R12 to R13, R13 to R14, R14 to R15, R15 to R16, R4 to R3, R6 to R7, R7 to R8, R8 to R9
Connections:
- net +9V: now also Q2.3 (D); no longer R2.1
- net GND: now also R2.2, R6.2
- net VGND: now reaches POT1.2, R11.1, R14.2, R3.2
- net VGND: now also J3.1 (Pin_1), R4.2; no longer R2.2
- net SEND: now reaches C2.1, J5.1 (Pin_1), R1.1
- net SEND: no longer J3.1 (Pin_1)
- net at J7.1 (Pin_1): now also C6.2
- net at J6.1 (Pin_1): now also R2.1, C3.1; no longer C6.2
- net at R8.1: now also C4.1
- new net: C3.2, Q2.1 (G), R4.1
- new net: C4.2, Q2.2 (S), R6.1
Other:
- note added: "エフェクトOUTのみPOTを通す"
- note added: "バッファがないとエフェクター先でバイパスされた時に短絡して原音に影響してしまう しかしBLENDERを使うときにエフェクタ先でバイパスにすることは無いはず"
- note removed: "MASTER"
- note removed: "コンデンサー前に1M入れたい"
- moved on the sheet: C2, C5, J5, POT1, Q1, R1, R14, R3, R5, R7, R8, R9
